File: hardware/cpu.kicad_sch (KiCad schematic)
At the start: 27 parts, among them J6 Conn_02x05_SWD, SW6 Switch_SW_Push, U2 RP2040, U3 W25Q128JVS, X1 12MHz

Commit message: hardware: pcb routing complete
Parts:
- renumbered C9 to C10, C10 to C11, C11 to C12, C12 to C13, C13 to C14, C14 to C15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
